File: logic_nixie_clock.kicad_pcb (KiCad board)
At the start: 2 copper layers, 186 x 45 mm, 232 parts, among them J1 Conn_01x03, Q1 MMBTA42, Q10 MMBTA42, Q11 MMBTA42, Q12 MMBTA42, Q13 MMBTA42, Q14 MMBTA42, Q15 MMBTA42, Q16 MMBTA42, Q17 MMBTA42, Q18 MMBTA42, Q19 MMBTA42, Q2 MMBTA42, Q20 MMBTA42, Q21 MMBTA42, Q22 MMBTA42, Q23 MMBTA42, Q24 MMBTA42, Q25 MMBTA42, Q26 MMBTA42, Q27 MMBTA42, Q28 MMBTA42, Q29 MMBTA42, Q3 MMBTA42, Q30 MMBTA42, Q31 MMBTA42, Q32 MMBTA42, Q33 MMBTA42, Q34 MMBTA42, Q35 MMBTA42, Q36 MMBTA42, Q37 MMBTA42, Q38 MMBTA42, Q39 MMBTA42, Q4 MMBTA42, Q40 MMBTA42, Q41 MMBTA42, Q42 MMBTA42, Q43 MMBTA42, Q44 MMBTA42, Q45 MMBTA42, Q46 MMBTA42, Q47 MMBTA42, Q48 MMBTA42, Q49 MMBTA42, Q5 MMBTA42, Q6 MMBTA42, Q7 MMBTA42, Q8 MMBTA42, Q9 MMBTA42, SW1 SW_Push, SW2 SW_Push, SW3 SW_Push, SW4 SW_Push, SW5 SW_Push, U1 4017, U10 4071, U11 4017, U12 4017, U13 4017, U14 4017, U15 40106, U17 4081, U2 4017, U21 4070, U3 4017, U4 4060, U5 4013, U9 4017, Y1 Crystal

Commit message: Rev 1.1
Parts:
- removed D3: D, Diode_SMD:D_MELF
- added D4: ABS10, Diode_SMD:Diode_Bridge_Diotec_ABS, F.Cu at (108.2, 45.2)
- added R15: 220k, Resistor_SMD:R_1206_3216Metric_Pad1.30x1.75mm_HandSolder, F.Cu at (114.8, 46.6)
- added R31: 220k, Resistor_SMD:R_1206_3216Metric_Pad1.30x1.75mm_HandSolder, F.Cu at (114.8, 41.5)
- D10, D9: value 4V7 -> 5V1
- R21: value 47 -> 220
- moved G*** 52.0 mm to (165.6, 46.6)
- moved TR2 35.4 mm to (76.0, 45.8), turned to 0 degrees
- moved R98 22.9 mm to (106.9, 69.9), turned to 0 degrees
- moved R95 10.4 mm to (101.4, 67.5), turned to 180 degrees
- moved R97 8.73 mm to (107.0, 60.5), turned to 90 degrees
- moved C16 6.71 mm to (63.1, 39.7), turned to 180 degrees
- moved R99 3.89 mm to (109.1, 50.8), turned to 180 degrees
- moved Q7 3.41 mm to (88.6, 47.1)
- moved R51 1.64 mm to (101.7, 54.9), turned to -90 degrees
- moved R64 1.63 mm to (111.3, 54.7)
- moved Q9 1.20 mm to (98.3, 50.7)
- moved U13 1.13 mm to (69.1, 43.3)
- moved C13 1.10 mm to (74.4, 40.2)
- moved R9 0.82 mm to (137.6, 72.7)
- moved R12 0.70 mm to (84.1, 39.5)
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Connections:
- TR2 pad 5: /LVAC -> Net-(D4-Pad3)
- TR2 pad 7: /LVAC -> GND
- TR2 pad 9: GND -> /LVAC
Routing:
- net GND: track 745.9 -> 793.8 mm, vias 24 -> 23
- net /LVAC: track 169.1 -> 138.5 mm
- net Net-(D4-Pad4): track 2.60 -> 32.3 mm, vias 0 -> 2
- net Net-(NE1-Pad2): track 19.3 -> 4.00 mm, vias 1 -> 0
- net /8_hr1: track 32.3 -> 40.6 mm, vias 2 -> 4
- net Net-(U13-Reset): track 110.0 -> 101.9 mm
- net /4_hr1: track 24.0 -> 31.6 mm
- net /1_hr1: track 81.4 -> 74.9 mm, vias 5 -> 3
- net /9_hr1: track 54.5 -> 59.9 mm, vias 3 -> 5
- net Net-(D4-Pad3): track 0.00 -> 5.30 mm
- net HT: track 241.6 -> 236.9 mm, vias 11 -> 10
- net nixie_gnd: track 512.0 -> 508.1 mm, vias 18 -> 22
- net Net-(NE2-Pad2): track 5.33 -> 8.83 mm
- net Net-(D10-K): track 59.8 -> 63.1 mm, vias 1 -> 3
- net /6_hr1_drv: track 6.67 -> 3.72 mm
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