File: logic_nixie_clock.kicad_sch (KiCad schematic)
At the start: 232 parts, among them J1 Conn_01x03, Q1 MMBTA42, Q10 MMBTA42, Q11 MMBTA42, Q12 MMBTA42, Q13 MMBTA42, Q14 MMBTA42, Q15 MMBTA42, Q16 MMBTA42, Q17 MMBTA42, Q18 MMBTA42, Q19 MMBTA42, Q2 MMBTA42, Q20 MMBTA42, Q21 MMBTA42, Q22 MMBTA42, Q23 MMBTA42, Q24 MMBTA42, Q25 MMBTA42, Q26 MMBTA42, Q27 MMBTA42, Q28 MMBTA42, Q29 MMBTA42, Q3 MMBTA42, Q30 MMBTA42, Q31 MMBTA42, Q32 MMBTA42, Q33 MMBTA42, Q34 MMBTA42, Q35 MMBTA42, Q36 MMBTA42, Q37 MMBTA42, Q38 MMBTA42, Q39 MMBTA42, Q4 MMBTA42, Q40 MMBTA42, Q41 MMBTA42, Q42 MMBTA42, Q43 MMBTA42, Q44 MMBTA42, Q45 MMBTA42, Q46 MMBTA42, Q47 MMBTA42, Q48 MMBTA42, Q49 MMBTA42, Q5 MMBTA42, Q6 MMBTA42, Q7 MMBTA42, Q8 MMBTA42, Q9 MMBTA42, SW1 SW_Push, SW2 SW_Push, SW3 SW_Push, SW4 SW_Push, SW5 SW_Push, U1 4017, U10 4071, U11 4017, U12 4017, U13 4017, U14 4017, U15 40106, U17 4081, U2 4017, U21 4070, U3 4017, U4 4060, U5 4013, U9 4017, Y1 Crystal

Commit message: Rev 1.1
Parts:
- removed D3: D, Diode_SMD:D_MELF, symbol Device:D
- added R15, R31: 220k, Resistor_SMD:R_1206_3216Metric_Pad1.30x1.75mm_HandSolder, symbol Device:R
- D10, D9: value 4V7 -> 5V1
Connections:
- net GND: now also R31.2
- net HT: now also R15.1
- net at TR2.1: now also D4.4; no longer D4.3
- net at TR2.5: now also D4.3; no longer D4.4
- new net: R15.2, R31.1
Other:
- note added: "Bleeder resistors"
- note added: "Blue text: 12 hr mode function "net" names derived from 24 hr Shifting outputs by one achieves 1-12 counting instead of 0-11"
- note added: "Clock inhibit blocks the mains clock to allow syncing to other clocks to below 1 Hz by holding the button just right"
- note added: "Decoupling caps and unused parts of ICs"
- note added: "Display drivers"
- note added: "Display tubes"
- note added: "For no leading zero on hours simply do not solder the Q12 transistor and R53 resistor R55 and Q14 can be omitted in 12hr clock"
- note added: "Jumper settings for 12/24h clocks: For 24h clock solder 0R in R10, R13, R30, R105, R107 and do not place R11, R12, R29, R104 For 12h clock solder 0R in R11, R12, R29, R104 and do not place R10, R13, R30, R105, R107 Default values shown for 24h clock"
- note added: "Load caps: For 12,5 pF crystal use 12 pF load capacitors Tuning might be needed"
- note added: "Mains frequency to 1 Hz divider"
- note added: "Neon indicators"
- note added: "Power supply"
- note added: "Solder R1 for 50 Hz, R2 for 60 Hz. Do not place the other resistor."
- note added: "TR1: 230V to 6V TR2: 6V to 230V For 120V mains use appropriate first transformer. 230V to 12 V should work, but it was not tested."
- note removed: "Blue text: 12 hr mode function "net" names derived from 24 hr Shifting outputs by one achieves 1-12 counting instead of 0-11 Solder R13 and R30 instead of R12 and R29 for 12h clock variant"
- note removed: "Clock inhibit blocks only mains clock to allow syncing to other clocks to below 1 Hz by holding the button just right"
- note removed: "For no leading zero on hours simply do not solder the Q12 transistor and R53 resistor 2_hr10 can be omitted in 12hr clock"
- note removed: "Load caps: For 6 pF crystal use 3.3 pF load capacitors Tuning might be needed"
- note removed: "Mains frequency to 1 Hz divider. Solder R1 for 50 Hz, R2 for 60 Hz"
- note removed: "TR1: 230V to 6V TR2: 10,5V to 230V This arrangement provides roughly 170VDC nominally"
- moved on the sheet: C12, C28, C8, NE1, NE2, NE3, NE4, NE5, NE6, Q1, Q10, Q12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
